File: Hardware/Production/SparkFun_GNSS_mosaic-G5_P3_panelized.kicad_pcb (KiCad board)
At the start: 4 copper layers, 115.8 x 100.6 mm, 575 parts, among them J1 USB_C_Receptacle, J10 U.FL, J2 Conn_01x06, J4 Conn_01x10, J5 SMA_Edge, J6 Conn_01x11, J8 JST_Locking_4, U1 DT1042-04SO, U2 RT9080-3.3, U3 mosaic-G5 P3

Commit message: Ready for protos
Parts:
- removed the ? at (129.6, 119.6) (x2)
- removed the ? at (227.7, 28.5) (x2)
- removed the ? at (129.6, 28.5) (x2)
- removed C2 (x4): 10uF, SparkFun-Capacitor:C_0603_1608Metric
- removed the Ref** at (175.9, 66.8)
- removed the Ref** at (227.2, 110.5)
- removed the Ref** at (227.2, 66.8)
- removed the TP3 at (150.5, 62.4)
- removed the TP3 at (201.8, 62.4)
- removed the TP3 at (201.8, 106.0)
- removed the TP4 at (150.5, 103.5)
- removed the TP4 at (201.8, 59.8)
- removed the TP4 at (201.8, 103.5)
- removed kibuzzard-6809429D (x4): G***, kibuzzard-6809429D
- removed kibuzzard-680942A9 (x4): G***, kibuzzard-680942A9
- removed the kibuzzard-68097087 at (208.5, 64.7)
- removed the kibuzzard-68097087 at (157.2, 64.7)
- removed the kibuzzard-68097087 at (208.5, 108.3)
- removed the kibuzzard-680973E5 at (201.8, 107.6)
- removed the kibuzzard-680973E5 at (150.5, 107.6)
- removed the kibuzzard-680973E5 at (201.8, 63.9)
- removed the kibuzzard-680973FC at (150.5, 102.1)
- removed the kibuzzard-680973FC at (150.5, 58.4)
- removed the kibuzzard-680973FC at (201.8, 102.1)
- added ?: , Fiducial_1mm_Mask3mm, F.Cu at (227.7, 28.5)
- added ?: , Fiducial_1mm_Mask3mm, F.Cu at (129.6, 28.5)
- added ?: , Fiducial_1.5mm_Mask3mm, F.Cu at (129.6, 119.6)
- added ?: , Fiducial_1.5mm_Mask3mm, B.Cu at (129.6, 119.6)
- added ?: , Fiducial_1mm_Mask3mm, B.Cu at (227.7, 28.5)
- added ?: , Fiducial_1mm_Mask3mm, B.Cu at (129.6, 28.5)
- added C14: 1.0uF, SparkFun-Capacitor:C_0603_1608Metric, F.Cu at (199.3, 94.6)
- added C14: 1.0uF, SparkFun-Capacitor:C_0603_1608Metric, F.Cu at (199.3, 50.9)
- added C14: 1.0uF, SparkFun-Capacitor:C_0603_1608Metric, F.Cu at (148.0, 50.9)
- added C14: 1.0uF, SparkFun-Capacitor:C_0603_1608Metric, F.Cu at (148.0, 94.6)
- added Ref**: Val**, SparkFun-Aesthetic:OSHW_Logo_4mm, B.Cu at (172.8, 68.1)
- added Ref**: Val**, SparkFun-Aesthetic:OSHW_Logo_4mm, B.Cu at (224.1, 68.1)
- added Ref**: Val**, SparkFun-Aesthetic:OSHW_Logo_4mm, B.Cu at (224.1, 111.8)
- added TP3: 1.0mm, SparkFun-Connector:TestPoint-1.0mm, B.Cu at (148.0, 62.4)
- added TP3: 1.0mm, SparkFun-Connector:TestPoint-1.0mm, B.Cu at (199.3, 106.0)
- added TP3: 1.0mm, SparkFun-Connector:TestPoint-1.0mm, B.Cu at (199.3, 62.4)
- added TP4: 1.0mm, SparkFun-Connector:TestPoint-1.0mm, B.Cu at (199.3, 103.5)
- added TP4: 1.0mm, SparkFun-Connector:TestPoint-1.0mm, B.Cu at (148.0, 59.8)
- added TP4: 1.0mm, SparkFun-Connector:TestPoint-1.0mm, B.Cu at (199.3, 59.8)
- added kibuzzard-68097087: G***, kibuzzard-68097087, B.Cu at (210.8, 65.9)
- added kibuzzard-68097087: G***, kibuzzard-68097087, B.Cu at (210.8, 109.6)
- added kibuzzard-68097087: G***, kibuzzard-68097087, B.Cu at (159.5, 65.9)
- added kibuzzard-680973E5: G***, kibuzzard-680973E5, B.Cu at (199.3, 107.6)
- added kibuzzard-680973E5: G***, kibuzzard-680973E5, B.Cu at (199.3, 63.9)
- added kibuzzard-680973E5: G***, kibuzzard-680973E5, B.Cu at (148.0, 63.9)
- added kibuzzard-680973FC: G***, kibuzzard-680973FC, B.Cu at (199.3, 58.3)
- added kibuzzard-680973FC: G***, kibuzzard-680973FC, B.Cu at (199.3, 102.0)
- added kibuzzard-680973FC: G***, kibuzzard-680973FC, B.Cu at (148.0, 58.3)
- added kibuzzard-680A6E0E: G***, kibuzzard-680A6E0E, F.Cu at (150.5, 77.9)
- added kibuzzard-680A6E0E: G***, kibuzzard-680A6E0E, F.Cu at (150.5, 34.2)
- added kibuzzard-680A6E0E: G***, kibuzzard-680A6E0E, F.Cu at (201.8, 34.2)
- added kibuzzard-680A6E0E: G***, kibuzzard-680A6E0E, F.Cu at (201.8, 77.9)
- added kibuzzard-680A6E23: G***, kibuzzard-680A6E23, B.Cu at (150.5, 34.0)
- added kibuzzard-680A6E23: G***, kibuzzard-680A6E23, B.Cu at (201.8, 34.0)
- added kibuzzard-680A6E23: G***, kibuzzard-680A6E23, B.Cu at (201.8, 77.7)
- added kibuzzard-680A6E23: G***, kibuzzard-680A6E23, B.Cu at (150.5, 77.7)
- added kibuzzard-680A7093: G***, kibuzzard-680A7093, B.Cu at (215.4, 64.0)
- added kibuzzard-680A7093: G***, kibuzzard-680A7093, B.Cu at (164.1, 64.0)
- added kibuzzard-680A7093: G***, kibuzzard-680A7093, B.Cu at (164.1, 107.7)
- added kibuzzard-680A7093: G***, kibuzzard-680A7093, B.Cu at (215.4, 107.7)
- added kibuzzard-680A70A3: G***, kibuzzard-680A70A3, B.Cu at (162.3, 64.0)
- added kibuzzard-680A70A3: G***, kibuzzard-680A70A3, B.Cu at (213.6, 107.7)
- added kibuzzard-680A70A3: G***, kibuzzard-680A70A3, B.Cu at (213.6, 64.0)
- added kibuzzard-680A70A3: G***, kibuzzard-680A70A3, B.Cu at (162.3, 107.7)
- added kibuzzard-680A70AF: G***, kibuzzard-680A70AF, B.Cu at (160.8, 64.0)
- added kibuzzard-680A70AF: G***, kibuzzard-680A70AF, B.Cu at (212.1, 64.0)
- added kibuzzard-680A70AF: G***, kibuzzard-680A70AF, B.Cu at (160.8, 107.7)
- added kibuzzard-680A70AF: G***, kibuzzard-680A70AF, B.Cu at (212.1, 107.7)
- added kibuzzard-680A70C6: G***, kibuzzard-680A70C6, B.Cu at (209.0, 64.0)
- added kibuzzard-680A70C6: G***, kibuzzard-680A70C6, B.Cu at (157.7, 107.7)
- added kibuzzard-680A70C6: G***, kibuzzard-680A70C6, B.Cu at (209.0, 107.7)
- added kibuzzard-680A70C6: G***, kibuzzard-680A70C6, B.Cu at (157.7, 64.0)
- C3 (x4): value 10uF -> 22uF
- TP1 (x4), TP3, TP4, TP5 (x4): value 1.25mm -> 1.0mm
- moved kibuzzard-680973FC 69.3 mm to (148.0, 102.0)
- moved kibuzzard-680973E5 43.8 mm to (148.0, 107.6)
- moved TP4 43.8 mm to (148.0, 103.5)
- moved TP5 43.7 mm to (145.4, 104.8)
- moved TP5 43.7 mm to (145.4, 61.1)
- moved Ref** 3.33 mm to (172.8, 111.8)
- moved kibuzzard-68097087 2.62 mm to (159.5, 109.6)
- moved TP3 2.54 mm to (148.0, 106.0)
Connections:
- TP3 pad 1: USB_D+ -> Net-(U1-I/O1)
- TP4 pad 1: USB_D- -> Net-(U1-I/O2)
Routing:
- net USB_D+: track 102.4 -> 94.1 mm
- net USB_D-: track 103.4 -> 95.1 mm
- net Net-(U1-I/O2): track 38.6 -> 43.0 mm, vias 0 -> 4
- net Net-(U1-I/O1): track 42.2 -> 46.3 mm, vias 0 -> 4
- net TX1: track 104.8 -> 108.2 mm
- net 3.3V: track 106.0 -> 109.1 mm
- net VUSB: track 209.8 -> 212.2 mm
- net RX1: track 114.7 -> 116.8 mm
- net Net-(D6-K): track 108.0 -> 107.2 mm
- net GND: vias 424 -> 448
