File: Hardware/Production/SparkFun_GNSS_mosaic-G5_P3_panelized.kicad_pcb (KiCad board)
At the start: 4 copper layers, 115.8 x 100.6 mm, 591 parts, among them J1 USB_C_Receptacle, J10 U.FL, J2 Conn_01x06, J4 Conn_01x10, J5 SMA_Edge, J6 Conn_01x11, J8 JST_Locking_4, U1 DT1042-04SO, U2 RT9080-3.3, U3 mosaic-G5 P3

Commit message: Re-panelized with paste reduction
Parts:
- removed the ? at (227.7, 28.5) (x2)
- removed the ? at (129.6, 28.5) (x2)
- removed the ? at (129.6, 119.6) (x2)
- removed the kibuzzard-6501FDDA at (199.9, 44.6)
- removed the kibuzzard-6501FDDA at (199.9, 88.3)
- removed the kibuzzard-6501FDDA at (148.6, 44.6)
- added ?: , Fiducial_1mm_Mask3mm, F.Cu at (227.7, 28.5)
- added ?: , Fiducial_1.5mm_Mask3mm, F.Cu at (129.6, 119.6)
- added ?: , Fiducial_1mm_Mask3mm, F.Cu at (129.6, 28.5)
- added ?: , Fiducial_1.5mm_Mask3mm, B.Cu at (129.6, 119.6)
- added ?: , Fiducial_1mm_Mask3mm, B.Cu at (129.6, 28.5)
- added ?: , Fiducial_1mm_Mask3mm, B.Cu at (227.7, 28.5)
- added kibuzzard-6501FDDA: G***, kibuzzard-6501FDDA, B.Cu at (199.9, 87.0)
- added kibuzzard-6501FDDA: G***, kibuzzard-6501FDDA, B.Cu at (148.6, 43.3)
- added kibuzzard-6501FDDA: G***, kibuzzard-6501FDDA, B.Cu at (199.9, 43.3)
- moved D14 67.4 mm to (173.3, 106.4)
- moved D14 67.4 mm to (224.6, 62.7)
- moved D3 67.4 mm to (173.3, 99.2)
- moved D3 67.4 mm to (224.6, 55.5)
- moved D8 67.4 mm to (203.1, 66.9)
- moved D8 67.4 mm to (151.8, 110.6)
- moved FID3 67.4 mm to (187.2, 31.2)
- moved FID3 67.4 mm to (135.9, 74.9)
- moved FID6 67.4 mm to (187.2, 31.2)
- moved FID6 67.4 mm to (135.9, 74.9)
- moved JP3 67.4 mm to (223.7, 39.5)
- moved JP3 67.4 mm to (172.4, 83.2)
- moved TR1 67.4 mm to (200.5, 61.1)
- moved TR1 67.4 mm to (149.2, 104.8)
- moved U3 67.4 mm to (160.7, 95.9)
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Connections:
- U3 pad 15: (no net) -> unconnected-(U3-Reserved-Pad15) (x4)
- U3 pad 16: (no net) -> unconnected-(U3-Reserved-Pad16) (x4)
- U3 pad 18: (no net) -> unconnected-(U3-Reserved-Pad18) (x4)
- U3 pad 19: (no net) -> unconnected-(U3-Reserved-Pad19) (x4)
- U3 pad 20: (no net) -> unconnected-(U3-Reserved-Pad20) (x4)
- U3 pad 22: (no net) -> unconnected-(U3-Reserved-Pad22) (x4)
- U3 pad 23: (no net) -> unconnected-(U3-Reserved-Pad23) (x4)
- U3 pad 24: (no net) -> unconnected-(U3-Reserved-Pad24) (x4)
- U3 pad 30: (no net) -> unconnected-(U3-Reserved-Pad30) (x4)
- U3 pad 31: (no net) -> unconnected-(U3-Reserved-Pad31) (x4)
- U3 pad 32: (no net) -> unconnected-(U3-Reserved-Pad32) (x4)
- U3 pad 33: (no net) -> unconnected-(U3-Reserved-Pad33) (x4)
- U3 pad 35: (no net) -> unconnected-(U3-Reserved-Pad35) (x4)
- U3 pad 36: (no net) -> unconnected-(U3-Reserved-Pad36) (x4)
- U3 pad 37: (no net) -> unconnected-(U3-Reserved-Pad37) (x4)
- U3 pad 38: (no net) -> unconnected-(U3-Reserved-Pad38) (x4)
- U3 pad 8: (no net) -> unconnected-(U3-Reserved-Pad8) (x4)
