File: Hardware/SparkFun_GNSS_mosaic-G5_P3.kicad_pcb (KiCad board)
At the start: 4 copper layers, 43.2 x 43.2 mm, 143 parts, among them J1 USB_C_Receptacle, J10 U.FL, J2 Conn_01x06, J4 Conn_01x10, J5 SMA_Edge, J6 Conn_01x11, J8 JST_Locking_4, U1 DT1042-04SO, U2 RT9080-3.3, U3 mosaic-G5 P3

Commit message: Ready for protos
Parts:
- removed C2: 10uF, SparkFun-Capacitor:C_0603_1608Metric
- removed kibuzzard-6809429D: G***, kibuzzard-6809429D
- removed kibuzzard-680942A9: G***, kibuzzard-680942A9
- added C14: 1.0uF, SparkFun-Capacitor:C_0603_1608Metric, F.Cu at (148.0, 94.6)
- added kibuzzard-680A6E0E: G***, kibuzzard-680A6E0E, F.Cu at (150.5, 77.9)
- added kibuzzard-680A6E23: G***, kibuzzard-680A6E23, B.Cu at (150.5, 77.7)
- added kibuzzard-680A7093: G***, kibuzzard-680A7093, B.Cu at (164.1, 107.7)
- added kibuzzard-680A70A3: G***, kibuzzard-680A70A3, B.Cu at (162.3, 107.7)
- added kibuzzard-680A70AF: G***, kibuzzard-680A70AF, B.Cu at (160.8, 107.7)
- added kibuzzard-680A70C6: G***, kibuzzard-680A70C6, B.Cu at (157.7, 107.7)
- C3: value 10uF -> 22uF
- TP1, TP3, TP4, TP5: value 1.25mm -> 1.0mm
- moved Ref** 3.33 mm to (172.8, 111.8)
- moved kibuzzard-68097087 2.62 mm to (159.5, 109.6)
- moved kibuzzard-680973FC 2.54 mm to (148.0, 102.0)
- moved TP3 2.54 mm to (148.0, 106.0)
- moved TP4 2.54 mm to (148.0, 103.5)
- moved kibuzzard-680973E5 2.54 mm to (148.0, 107.6)
Connections:
- TP3 pad 1: USB_D+ -> Net-(U1-I/O1)
- TP4 pad 1: USB_D- -> Net-(U1-I/O2)
Routing:
- net USB_D+: track 25.6 -> 23.5 mm
- net USB_D-: track 25.8 -> 23.8 mm
- net Net-(U1-I/O2): track 9.66 -> 10.8 mm, vias 0 -> 1
- net Net-(U1-I/O1): track 10.5 -> 11.6 mm, vias 0 -> 1
- net TX1: track 26.2 -> 27.1 mm
- net 3.3V: track 26.5 -> 27.3 mm
- net VUSB: track 52.4 -> 53.0 mm
- net RX1: track 28.7 -> 29.2 mm
- net GND: vias 106 -> 112

Commit message: Re-panelized with paste reduction
Parts:
- moved kibuzzard-6501FDDA 1.27 mm to (148.6, 87.0)
Connections:
- U3 pad 15: (no net) -> unconnected-(U3-Reserved-Pad15)
- U3 pad 16: (no net) -> unconnected-(U3-Reserved-Pad16)
- U3 pad 18: (no net) -> unconnected-(U3-Reserved-Pad18)
- U3 pad 19: (no net) -> unconnected-(U3-Reserved-Pad19)
- U3 pad 20: (no net) -> unconnected-(U3-Reserved-Pad20)
- U3 pad 22: (no net) -> unconnected-(U3-Reserved-Pad22)
- U3 pad 23: (no net) -> unconnected-(U3-Reserved-Pad23)
- U3 pad 24: (no net) -> unconnected-(U3-Reserved-Pad24)
- U3 pad 30: (no net) -> unconnected-(U3-Reserved-Pad30)
- U3 pad 31: (no net) -> unconnected-(U3-Reserved-Pad31)
- U3 pad 32: (no net) -> unconnected-(U3-Reserved-Pad32)
- U3 pad 33: (no net) -> unconnected-(U3-Reserved-Pad33)
- U3 pad 35: (no net) -> unconnected-(U3-Reserved-Pad35)
- U3 pad 36: (no net) -> unconnected-(U3-Reserved-Pad36)
- U3 pad 37: (no net) -> unconnected-(U3-Reserved-Pad37)
- U3 pad 38: (no net) -> unconnected-(U3-Reserved-Pad38)
- U3 pad 8: (no net) -> unconnected-(U3-Reserved-Pad8)

Commit message: Update symbols and 3D models
Parts:
- J10: value U.FL -> Val**
- J2: footprint SparkFun-Connector:1x06 -> SparkFun-Connector:1x06_P2.54mm
- J4: footprint SparkFun-Connector:1x10 -> SparkFun-Connector:1x10_P2.54mm
- J5: footprint SparkFun-Connector:SMA_Edge -> SparkFun-Connector:SMA_Edge_6.3mm
- J6: footprint SparkFun-Connector:1x11 -> SparkFun-Connector:1x11_P2.54mm
- J8: footprint SparkFun-Connector:JST_SMD_1.25mm-4_Locking -> SparkFun-Connector:JST_1x04_P1.25mm_Locking_Horizontal_SMD
- TR1: footprint SparkFun-Coil:RFCMF1220100M4T -> SparkFun-Coil:Choke_100MHz_USB
- U3: footprint SparkFun-CustomParts:MOSAIC-G5_LGA54 -> SparkFun-GPS:MOSAIC-G5_LGA54
Connections:
- TR1 pad 1: Net-(U1-I/O2) -> unconnected-(TR1-Pad1)
- TR1 pad 2: USB_D- -> unconnected-(TR1-Pad2)
- TR1 pad 3: Net-(U1-I/O1) -> (no net)
- TR1 pad 4: USB_D+ -> (no net)
Changed lines of the file:
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@@
 	(net 74 "unconnected-(U3-Reserved-Pad31)")
 	(net 75 "unconnected-(U3-Reserved-Pad19)")
+	(net 76 "unconnected-(TR1-Pad1)")
+	(net 77 "unconnected-(TR1-Pad2)")
 	(footprint "kibuzzard-68094456"
 		(layer "F.Cu")
@@
 		(embedded_fonts no)
 	)
-	(footprint "SparkFun-Connector:1x06"
+	(footprint "SparkFun-Connector:1x06_P2.54mm"
 		(layer "F.Cu")
 		(at 143.51 80.645 -90)
@@
 			(remove_unused_layers yes)
 			(keep_end_layers yes)
-			(zone_layer_connections "In1.Cu")
+			(zone_layer_connections)
 			(net 1 "GND")
 			(pinfunction "Pin_6")
@@
 		(fp_poly
 			(pts
+				(xy -3.425 0.84) (xy -3.025 0.84) (xy -3.025 -0.16) (xy -3.425 -0.16)
+			)
+			(stroke
+				(width 0)
+				(type default)
+			)
+			(fill yes)
+			(layer "F.Paste")
+		)
+		(fp_poly
+			(pts
+				(xy -2.65 0.84) (xy -2.25 0.84) (xy -2.25 -0.16) (xy -2.65 -0.16)
+			)
+			(stroke
+				(width 0)
+				(type default)
+			)
+			(fill yes)
+			(layer "F.Paste")
+		)
+		(fp_poly
+			(pts
+				(xy 2.25 0.84) (xy 2.65 0.84) (xy 2.65 -0.16) (xy 2.25 -0.16)
+			)
+			(stroke
+				(width 0)
+				(type default)
+			)
+			(fill yes)
+			(layer "F.Paste")
+		)
+		(fp_poly
+			(pts
+				(xy 3.025 0.84) (xy 3.425 0.84) (xy 3.425 -0.16) (xy 3.025 -0.16)
+			)
+			(stroke
+				(width 0)
+				(type default)
+			)
+			(fill yes)
+			(layer "F.Paste")
+		)
+		(fp_poly
+			(pts
 				(xy -4.9 -0.25) (xy 4.9 -0.25) (xy 4.9 2.05) (xy 4.5 2.05) (xy 4.5 4.2) (xy 4.9 4.2) (xy 4.9 5.95)
 				(xy 4.5 5.95) (xy 4.5 7.85) (xy -4.5 7.85) (xy -4.5 5.95) (xy -4.9 5.95) (xy -4.9 4.2) (xy -4.5 4.2)
@@
 			(at -3.225 0.34 90)
 			(size 0.6 1)
-			(layers "F.Cu" "F.Mask" "F.Paste")
+			(layers "F.Cu" "F.Mask")
 			(net 1 "GND")
 			(pinfunction "GND")
@@
 			(at 3.225 0.34 270)
 			(size 0.6 1)
-			(layers "F.Cu" "F.Mask" "F.Paste")
+			(layers "F.Cu" "F.Mask")
 			(net 1 "GND")
 			(pinfunction "GND")
@@
 			(at -2.45 0.34 90)
 			(size 0.6 1)
-			(layers "F.Cu" "F.Mask" "F.Paste")
+			(layers "F.Cu" "F.Mask")
 			(net 4 "VUSB")
 			(pinfunction "VBUS")
@@
 			(at 2.45 0.34 270)
 			(size 0.6 1)
-			(layers "F.Cu" "F.Mask" "F.Paste")
+			(layers "F.Cu" "F.Mask")
 			(net 4 "VUSB")
 			(pinfunction "VBUS")
@@
 		(model "${SPARKFUN_KICAD_LIBRARY}/Footprints/SparkFun-3D-models/Connector/USB-C_16.step"
 			(offset
-				(xyz 0 -5 0)
+				(xyz 0 -5.13 0)
 			)
 			(scale
@@
 			)
 			(rotate
-				(xyz -90 0 0)
+				(xyz -90 -0 -0)
 			)
 		)
@@
 		(embedded_fonts no)
 	)
-	(footprint "SparkFun-Connector:JST_SMD_1.25mm-4_Locking"
+	(footprint "SparkFun-Connector:JST_1x04_P1.25mm_Locking_Horizontal_SMD"
 		(layer "F.Cu")
 		(at 138.404 86.995 -90)
@@
 			)
 		)
-		(property "Datasheet" "https://docs.broadcom.com/docs/AV02-0551EN"
+		(property "Datasheet" "https://www.kingbrightusa.com/images/catalog/SPEC/APT1608SURCK.pdf"
 			(at 0 0 90)
 			(unlocked yes)
@@
 		(embedded_fonts no)
 	)
-	(footprint "SparkFun-Connector:SMA_Edge"
+	(footprint "SparkFun-Connector:SMA_Edge_6.3mm"
 		(layer "F.Cu")
 		(at 176.11215 99.695 -90)
@@
 			)
 		)
-		(property "Datasheet" "https://www.sparkfun.com/datasheets/Wireless/Antenna/SMA-Connector.pdf"
+		(property "Datasheet" "https://cdn.sparkfun.com/assets/4/1/2/2/0/SMA-Connector.pdf"
 			(at 0 0 270)
 			(unlocked yes)
@@
 			)
 		)
-		(property "Description" "SMA PCB Edge Mount connector"
+		(property "Description" "Not for new designs. Use 8mm variant. SMA PCB Edge Mount connector"
 			(at 0 0 270)
 			(unlocked yes)
@@
 		)
 	)
-	(footprint "SparkFun-Coil:RFCMF1220100M4T"
+	(footprint "SparkFun-Coil:Choke_100MHz_USB"
 		(layer "F.Cu")
 		(at 149.225 104.775)
-		(tags "SparkFun")
+		(descr "RFCMF1220100M4T")
+		(tags "SparkFun USB Transformer Choke")
 		(property "Reference" "TR1"
 			(at 0 -1.3 0)
@@
 			(size 0.9 0.4)
 			(layers "F.Cu" "F.Mask" "F.Paste")
-			(net 18 "Net-(U1-I{slash}O2)")
+			(net 76 "unconnected-(TR1-Pad1)")
 			(pintype "passive")
 			(thermal_bridge_angle 0)
@@
 			(size 0.9 0.4)
 			(layers "F.Cu" "F.Mask" "F.Paste")
-			(net 12 "USB_D-")
+			(net 77 "unconnected-(TR1-Pad2)")
 			(pintype "passive")
 			(thermal_bridge_angle 0)
@@
 			(size 0.9 0.4)
 			(layers "F.Cu" "F.Mask" "F.Paste")
-			(net 8 "Net-(U1-I{slash}O1)")
-			(pintype "passive")
 			(thermal_bridge_angle 0)
 		)
@@
 			(size 0.9 0.4)
 			(layers "F.Cu" "F.Mask" "F.Paste")
-			(net 10 "USB_D+")
-			(pintype "passive")
 			(thermal_bridge_angle 0)
 		)
 		(embedded_fonts no)
-		(model "${SPARKFUN_KICAD_LIBRARY}/Footprints/SparkFun-3D-models/Coil/CHIP_100M4T_WAL.step"
+		(model "${SPARKFUN_KICAD_LIBRARY}/Footprints/SparkFun-3D-models/Coil/Choke_100MHz_USB_RFCMF1220100M4T.stp"
 			(offset
-				(xyz 0 0 0)
+				(xyz 0 0 -0.02)
 			)
 			(scale
-				(xyz 1 0.9 0.9)
+				(xyz 1 1 1)
 			)
 			(rotate
-				(xyz 0 0 0)
+				(xyz -90 -0 -0)
 			)
 		)
@@
 			)
 		)
-		(property "Value" "U.FL"
+		(property "Value" "Val**"
 			(at 0 2.2 180)
 			(layer "F.Fab")
@@
 		)
 	)
-	(footprint "SparkFun-Connector:1x11"
+	(footprint "SparkFun-Connector:1x11_P2.54mm"
 		(layer "F.Cu")
 		(at 145.415 75.565)
@@
 			(remove_unused_layers yes)
 			(keep_end_layers yes)
-			(zone_layer_connections "In1.Cu")
+			(zone_layer_connections)
 			(net 1 "GND")
 			(pinfunction "Pin_1")
@@
 			(remove_unused_layers yes)
 			(keep_end_layers yes)
-			(zone_layer_connections "In2.Cu")
+			(zone_layer_connections)
 			(net 7 "3.3V")
 			(pinfunction "Pin_2")
@@
 			(remove_unused_layers yes)
 			(keep_end_layers yes)
-			(zone_layer_connections "In1.Cu")
+			(zone_layer_connections)
 			(net 1 "GND")
 			(pinfunction "Pin_11")
@@
 		)
 	)
-	(footprint "SparkFun-Connector:1x10"
+	(footprint "SparkFun-Connector:1x10_P2.54mm"
 		(layer "F.Cu")
 		(at 145.415 116.205)
@@
 			(remove_unused_layers yes)
 			(keep_end_layers yes)
-			(zone_layer_connections "In1.Cu")
+			(zone_layer_connections)
 			(net 1 "GND")
 			(pinfunction "Pin_1")
@@
 			(remove_unused_layers yes)
 			(keep_end_layers yes)
-			(zone_layer_connections "In2.Cu")
+			(zone_layer_connections)
 			(net 7 "3.3V")
 			(pinfunction "Pin_2")
@@
 			(remove_unused_layers yes)
 			(keep_end_layers yes)
-			(zone_layer_connections "In1.Cu")
+			(zone_layer_connections)
 			(net 1 "GND")
 			(pinfunction "Pin_10")
@@
 		)
 		(group ""
-			(members "0d812ac4-45c5-4074-a21d-a15c986d1593" "2aa57e34-aab1-4718-b10c-e7bf749cab3e"
-				"4e8955c2-d4d5-4d20-892b-c3bd71070fa4" "62ff28fd-e231-4183-9428-a66c189cafb9"
-				"8fc7f299-86f8-47a4-845c-6d2ecc958675" "ba07f525-b9e3-4cb0-a990-bc904591ca9a"
-				"d01ecb04-ec88-49f3-801a-6970698ae975" "daacec4b-f899-4241-84e8-c56dd70fb1f5"
-				"e57c7f8d-c5b6-450a-b33d-8ed1ef673eb7"
+			(members "0319149b-0508-46fe-b10e-db00a96ee328" "1ffd76ad-8d67-428d-8c88-842be30300e3"
+				"3341c00e-af62-477e-8247-a9b343a50169" "5e24fde4-e343-4f70-98f5-d8caf7180338"
+				"72a2c5f9-dae3-4b73-8bbe-cce428158150" "aebf9088-5a70-4eb7-8803-386492437048"
+				"cafb3518-068e-414c-adce-5e5b61885111" "d73928a2-3b5b-4192-9fc9-4eecae7c22e5"
+				"d874976a-ef91-431b-9886-e883b595db5b"
 			)
 		)
@@
 		(embedded_fonts no)
 	)
-	(footprint "SparkFun-CustomParts:MOSAIC-G5_LGA54"
+	(footprint "SparkFun-GPS:MOSAIC-G5_LGA54"
 		(layer "F.Cu")
 		(at 160.655 95.885 180)
-		(tags "SparkFun mosaic-G5 LGA")
+		(descr "Septentrio mosaic-G5 GNSS Receiver")
+		(tags "SparkFun GNSS GPS Receiver mosaic-G5 LGA")
 		(property "Reference" "U3"
 			(at 0 -12.5 180)
@@
 		)
 		(embedded_fonts no)
-		(model "C:/Users/pc235/Documents/GitHub/SparkFun_GNSS_Flex_Modules/Documents/mosaic-G5.step"
+		(model "${SPARKFUN_KICAD_LIBRARY}/Footprints/SparkFun-3D-models/GPS/mosaic-G5.step"
 			(offset
 				(xyz -8.2 11.4 0.8)
@@
 		)
 		(group ""
-			(members "2bb1b82f-3f5a-4277-9086-e94fe126cd6e" "67c6a02b-0e5a-43e2-b67d-f82086e74495"
-				"6f8a8646-8573-4471-9395-1825d4f0e738" "92d0a676-3a53-48a5-8950-5a0a8748f7b5"
-				"a6387d57-e6e1-4f52-8632-dfd0c7bed5fb" "aa59a7d7-35e9-4012-8fb3-9f79c031ba58"
-				"b090ac07-f671-421c-a4fc-87e7403bdc7d" "c093d747-ab78-449c-b866-793c52c7ff0b"
-				"e20ec5a6-6a4f-43b0-80fd-333608d5763c"
+			(members "014f352c-6644-4d01-9fd3-03adeccc1082" "0d0ec3a6-0ff4-4b8c-9b06-57d2e7684e27"
+				"22fbebb5-04de-48ea-897a-d5974b004bb5" "23843b0c-a701-4538-8086-b300b39572bc"
+				"5643d08b-6c06-48a3-9e41-a71877045e1c" "67965c25-9c13-43ce-a0fd-2becff749b95"
+				"c9c0d9ae-0b72-4702-883f-0a5f86348c8b" "d0f11a22-ef0b-4099-a730-7036029a3e6d"
+				"d5ca484b-b390-440a-b5e6-21e7864f038b"
 			)
 		)
@@
 		)
 		(group ""
-			(members "b952ecf6-98a6-42be-8443-3ebfce94549c")
+			(members "1c0ca3ba-5366-45f1-a53b-0b9228ad2ac2")
 		)
 		(embedded_fonts no)

Commit message: Fix RFCMF1220100M4T pin numbering
Connections:
- TR1 pad 1: unconnected-(TR1-Pad1) -> Net-(U1-I/O2)
- TR1 pad 2: unconnected-(TR1-Pad2) -> USB_D-
- TR1 pad 3: (no net) -> Net-(U1-I/O1)
- TR1 pad 4: (no net) -> USB_D+
Changed lines of the file:
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@@
 	(net 74 "unconnected-(U3-Reserved-Pad31)")
 	(net 75 "unconnected-(U3-Reserved-Pad19)")
-	(net 76 "unconnected-(TR1-Pad1)")
-	(net 77 "unconnected-(TR1-Pad2)")
 	(footprint "kibuzzard-68094456"
 		(layer "F.Cu")
@@
 			(size 0.9 0.4)
 			(layers "F.Cu" "F.Mask" "F.Paste")
-			(net 76 "unconnected-(TR1-Pad1)")
+			(net 18 "Net-(U1-I{slash}O2)")
 			(pintype "passive")
 			(thermal_bridge_angle 0)
@@
 			(size 0.9 0.4)
 			(layers "F.Cu" "F.Mask" "F.Paste")
-			(net 77 "unconnected-(TR1-Pad2)")
+			(net 12 "USB_D-")
 			(pintype "passive")
 			(thermal_bridge_angle 0)
@@
 			(size 0.9 0.4)
 			(layers "F.Cu" "F.Mask" "F.Paste")
+			(net 8 "Net-(U1-I{slash}O1)")
+			(pintype "passive")
 			(thermal_bridge_angle 0)
 		)
@@
 			(size 0.9 0.4)
 			(layers "F.Cu" "F.Mask" "F.Paste")
+			(net 10 "USB_D+")
+			(pintype "passive")
 			(thermal_bridge_angle 0)
 		)
@@
 		)
 		(group ""
-			(members "0319149b-0508-46fe-b10e-db00a96ee328" "1ffd76ad-8d67-428d-8c88-842be30300e3"
-				"3341c00e-af62-477e-8247-a9b343a50169" "5e24fde4-e343-4f70-98f5-d8caf7180338"
-				"72a2c5f9-dae3-4b73-8bbe-cce428158150" "aebf9088-5a70-4eb7-8803-386492437048"
-				"cafb3518-068e-414c-adce-5e5b61885111" "d73928a2-3b5b-4192-9fc9-4eecae7c22e5"
-				"d874976a-ef91-431b-9886-e883b595db5b"
+			(members "444f20df-3ae7-4255-8e86-d121584a48ba" "629e7c09-2d44-4827-90e2-e88f5e2ac0c7"
+				"6d1e3958-9067-4d58-bb5e-507ee88e3e2e" "7615b2a4-d265-4ee5-9c36-2b200ea7c3a7"
+				"77d0e5b4-f164-438c-bc56-19346ec023ab" "b11e193b-cd92-4f83-89de-7bed8d0d30da"
+				"b3ac6607-1dc7-403b-9119-255adc294e17" "c1763f8d-186e-4eae-8cd8-c8b677e23245"
+				"e703d786-2cdb-4385-be3a-1cda74546ccb"
 			)
 		)
@@
 		)
 		(group ""
-			(members "014f352c-6644-4d01-9fd3-03adeccc1082" "0d0ec3a6-0ff4-4b8c-9b06-57d2e7684e27"
-				"22fbebb5-04de-48ea-897a-d5974b004bb5" "23843b0c-a701-4538-8086-b300b39572bc"
-				"5643d08b-6c06-48a3-9e41-a71877045e1c" "67965c25-9c13-43ce-a0fd-2becff749b95"
-				"c9c0d9ae-0b72-4702-883f-0a5f86348c8b" "d0f11a22-ef0b-4099-a730-7036029a3e6d"
-				"d5ca484b-b390-440a-b5e6-21e7864f038b"
+			(members "4f79e22c-f852-444d-9f15-f7c9f548b855" "547ef769-8611-43a4-91f1-e6b637e9217e"
+				"75e388ff-ccec-4181-9dd7-73617f8aadda" "96035aff-3db5-47aa-a2e7-6f1ca22ea4c5"
+				"9eaf33dc-dddd-4ccf-99dc-72648b92f5d2" "b50c73e4-92f1-478b-82bc-b54e53092b1e"
+				"d3740f85-8de4-4fc2-bffd-84e54d5b7317" "df0fd15d-aa42-40ce-bcaf-6754cf276d72"
+				"ea85bbc0-e31a-4532-816f-6fc44d71f776"
 			)
 		)
@@
 		)
 		(group ""
-			(members "1c0ca3ba-5366-45f1-a53b-0b9228ad2ac2")
+			(members "fe83de5b-55ae-4aa6-8359-e9610166170f")
 		)
 		(embedded_fonts no)

Commit message: Update to latest SparkFun KiCad Libraries
Parts:
- J10: value Val** -> U.FL
- JP4: value ~ -> VSEL
- L1: value 470Ohm -> 470 Ohm
- REF.1: value ~ -> REF
- U3: footprint SparkFun-GPS:MOSAIC-G5_LGA54 -> SparkFun-GNSS:Septentrio_mosaic-G5_LGA54
- VREF.1: value ~ -> VREF
